File: schematic/laser_drawer.kicad_pcb (KiCad board)
At the start: 2 copper layers, 136.5 x 76.2 mm, 71 parts, among them P1 Xin, P2 Yin, P3 Rin, P4 Gin, P5 Bin, P6 Power, P7 SUB-D25 FC, U1 NE5532, U2 NE5532, U3 NE5532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

Commit message: update schematics
Connections:
- P7 pad 17: N-0000044 -> N-0000025
- P7 pad 4: N-0000049 (its old number) -> N-0000025
Routing:
- net N-0000025: track 0.00 -> 3.12 mm
