File: schematic/laser_drawer.sch (KiCad schematic (older format))
At the start: 71 parts, among them P1 Xin, P2 Yin, P3 Rin, P4 Gin, P5 Bin, P6 Power, P7 SUB-D25 FC, U1 NE5532, U2 NE5532, U3 NE5532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

Commit message: update schematics
Connections:
- wire segments 147 -> 150
- no-connect marks 14 -> 12
Changed lines of the file:
@@
-EESchema Schematic File Version 2  date Sat 11 May 2013 13:52:43 CEST
+EESchema Schematic File Version 2
 LIBS:power
 LIBS:device
@@
 	0    1    1    0
 $EndComp
-NoConn ~ 6350 2450
 NoConn ~ 6350 2850
 NoConn ~ 6350 2950
@@
 NoConn ~ 6350 3250
 NoConn ~ 6350 3350
-NoConn ~ 6350 3750
 NoConn ~ 6350 4150
 NoConn ~ 6350 4250
@@
 Text Label 6200 9200 1    60   ~ 0
 Vin
+Wire Wire Line
+	6350 2450 5900 2450
+Wire Wire Line
+	5900 2450 5900 3750
+Wire Wire Line
+	5900 3750 6350 3750
 $EndSCHEMATC
